Commit message: Modify model to prevent Lidar error

File: src/turtlebot3_description/urdf/turtlebot3_waffle.urdf.xacro (robot description, xacro)
@@ -25,4 +25,5 @@
   <link name="base_link">
     <visual>
+      <transparency>1</transparency>
       <origin xyz="-0.064 0 0.0" rpy="0 0 0"/>
       <geometry>
@@ -63,4 +64,5 @@
       </geometry>
       <material name="orange"/>
+      <transparency>1</transparency>
     </visual>
     <inertial>
@@ -242,5 +244,5 @@
     <parent link="base_link"/>
     <child link="base_scan"/>
-    <origin xyz="-0.064 0 0.122" rpy="0 0 0"/>
+    <origin xyz="-0.064 0 0.272" rpy="0 0 0"/> <!--0.122" rpy="0 0 0"/>-->
   </joint>
   <link name="base_scan">
@@ -253,5 +255,5 @@
     </visual>
     <collision>
-      <origin xyz="0.015 0 -0.0065" rpy="0 0 0"/>
+      <origin xyz="0.015 0 -0.0000" rpy="0 0 0"/><!--0.0065-->
       <geometry>
         <cylinder length="0.0315" radius="0.055"/>
